File: Rpi_RGB-LED_Shield_v1.kicad_pcb (KiCad board)
At the start: 2 copper layers, 65 x 56.5 mm, 33 parts, among them J1 RapberryPi_Conn, J2 ExpansionBoard_Conn, J3 PWR_Conn, J4 SerialConsole_Conn, U1 SN74LV4T125, U2 SN74LV4T125, U3 SN74LV4T125, U4 SN74LV4T125

Commit message: Push more effort
Parts:
- removed J4: SerialConsole_Conn, Connector_PinHeader_2.54mm:PinHeader_1x04_P2.54mm_Vertical
- moved R1 83.7 mm to (126.8, 106.0), turned to 180 degrees
- moved R2 76.8 mm to (131.2, 106.0)
- moved C11 71.7 mm to (143.0, 87.8), turned to 180 degrees
- moved C10 68.4 mm to (143.0, 89.2), turned to 180 degrees
- moved R3 66.9 mm to (140.8, 106.0), turned to 180 degrees
- moved R10 60.0 mm to (143.0, 92.2)
- moved R4 60.0 mm to (145.2, 106.0)
- moved R5 47.6 mm to (154.8, 106.0), turned to 180 degrees
- moved R11 45.6 mm to (143.0, 90.8)
- moved C2 36.7 mm to (129.2, 115.2), turned to 180 degrees
- moved R6 31.8 mm to (159.2, 106.0)
- moved C6 30.8 mm to (129.2, 113.8), turned to 180 degrees
- moved C7 30.0 mm to (143.0, 113.8), turned to 180 degrees
- moved C3 28.6 mm to (143.0, 115.2), turned to 180 degrees
- moved C8 21.4 mm to (157.0, 113.8), turned to 180 degrees
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Connections:
- J2 pad 10: GND -> MOSI_1
- J2 pad 11: SCK_1 -> GND
- J2 pad 12: GND -> SCK_1
- J2 pad 13: MOSI_2 -> GND
- J2 pad 14: GND -> MOSI_2
- J2 pad 15: SCK_2 -> GND
- J2 pad 16: GND -> SCK_2
- J2 pad 17: MOSI_3 -> GND
- J2 pad 18: GND -> MOSI_3
- J2 pad 19: SCK_3 -> GND
- J2 pad 20: GND -> SCK_3
- J2 pad 5: MOSI_0 -> GND
- J2 pad 6: GND -> MOSI_0
- J2 pad 7: SCK_0 -> GND
- J2 pad 8: GND -> SCK_0
- J2 pad 9: MOSI_1 -> GND
- R7 pad 2: GPIO20 -> GPIO26
- U4 pad 1: GPIO20 -> GPIO26
- U4 pad 4: GPIO20 -> GPIO26
Routing:
- net VCC: track 0.00 -> 114.8 mm, vias 0 -> 1
- net GPIO5: track 0.00 -> 58.7 mm
- net GPIO12: track 0.00 -> 49.9 mm
- net GPIO6: track 0.00 -> 49.2 mm
- net SCK: track 0.00 -> 47.8 mm
- net GPIO21: track 0.00 -> 38.8 mm
- net GPIO16: track 0.00 -> 37.9 mm
- net GPIO13: track 0.00 -> 37.1 mm
- net GPIO26: track 0.00 -> 34.5 mm
- net GPIO19: track 0.00 -> 25.0 mm
- net SCK_7: track 0.00 -> 24.7 mm
- net MOSI_7: track 0.00 -> 23.7 mm
- net MOSI: track 0.00 -> 22.1 mm
- net SCK_5: track 0.00 -> 21.1 mm
- net MOSI_5: track 0.00 -> 20.7 mm
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- added copper zone on F.Cu, net VCC
Other:
- board text added: "+"
- board text added: "-"
- board text added: "5V ONLY"
- board text added: "PWR"

Commit message: A little bit closer to the final
Parts:
- moved R9 4.16 mm to (119.8, 103.0), turned to 90 degrees
- moved C10 3.25 mm to (144.2, 92.2)
- moved D1 2.46 mm to (119.8, 100.0), turned to 270 degrees
- moved R10 1.95 mm to (144.2, 90.8)
- moved R11 1.95 mm to (144.2, 89.2)
- moved C11 1.25 mm to (144.2, 87.8)
- moved C6 1.25 mm to (128.2, 114.5), turned to 270 degrees
- moved C3 1.06 mm to (143.8, 114.5), turned to 270 degrees
- moved C4 1.06 mm to (157.8, 114.5), turned to 270 degrees
- moved C5 1.06 mm to (171.8, 114.5), turned to 270 degrees
- moved C7 1.06 mm to (142.2, 114.5), turned to 270 degrees
- moved C8 1.06 mm to (156.2, 114.5), turned to 270 degrees
- moved C9 1.06 mm to (170.2, 114.5), turned to 270 degrees
- moved C2 0.90 mm to (129.8, 114.5), turned to 270 degrees
Connections:
- J1 pad 1: +3V3 -> Net-(J1-Pad1)
- J1 pad 17: +3V3 -> Net-(J1-Pad17)
- J2 pad 2: GND -> VCC
- J2 pad 38: VCC -> GND
- J2 pad 4: GND -> VCC
- J2 pad 40: VCC -> GND
Routing:
- net MOSI: track 22.1 -> 140.4 mm, vias 0 -> 8
- net VCC: track 114.8 -> 226.8 mm, vias 1 -> 9
- net SCK: track 47.8 -> 141.0 mm, vias 0 -> 8
- net GPIO19: track 25.0 -> 36.4 mm
- net GPIO6: track 49.2 -> 60.5 mm
- net GPIO21: track 38.8 -> 50.2 mm
- net GPIO13: track 37.1 -> 48.5 mm
- net SCK_0: track 8.88 -> 18.8 mm
- net MOSI_0: track 11.4 -> 18.8 mm
- net GPIO26: track 34.5 -> 39.2 mm
- net GPIO16: track 37.9 -> 42.6 mm
- net GPIO12: track 49.9 -> 54.7 mm
- net GPIO5: track 58.7 -> 62.9 mm
- net SCK_6: track 15.8 -> 19.8 mm
- net SCK_3: track 18.0 -> 14.1 mm
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Other:
- outline, holes or cut-outs redrawn
- board text added: "INGARAGE ASSISTIVE TECHNOLOGY CO."
- board text added: "RGB LED STRIP RASPBERRY-PI HAT"
