File: Rpi_RGB-LED_Shield_v1.sch (KiCad schematic (older format))
At the start: 3 parts

Commit message: Put some progress
Parts:
- added C1: 100uF, symbol Device:CP1_Small
- added C2, C3, C4, C5: 1uF, Capacitor_SMD:C_0603_1608Metric, symbol Device:C_Small
- added C6, C7, C8, C9: 0.1uF, Capacitor_SMD:C_0603_1608Metric, symbol Device:C_Small
- added C?: 1uF, symbol Device:C_Small
- added C?: 0.1uF, symbol Device:C_Small
- added D1: LED, LED_SMD:LED_0603_1608Metric, symbol Device:LED
- added J3: Screw_Terminal_01x02, symbol Connector:Screw_Terminal_01x02
- added R1, R2, R3, R4, R5, R6, R7, R8: 10K, Resistor_SMD:R_0201_0603Metric, symbol Device:R_Small
- added R9: 1K, Resistor_SMD:R_0201_0603Metric, symbol Device:R_Small
- added U2, U3, U4: SN74LV4T125, symbol InGarage_Logic_LevelTranslator:SN74LV4T125
- gave numbers to parts that had none: 3
Connections:
- net +3V3: now also J1.17 (Pin_17)
- net GND: now also C1.2, C2.2, C3.2, C4.2, C5.2, C6.2, C7.2, C8.2, C9.2, C?.2, C?.2, D1.1 (K), J3.1 (Pin_1), U2.7 (GND), U3.7 (GND), U4.7 (GND)
- net MOSI_0: now also U1.3 (1Y)
- net MOSI_1: now also U1.8 (3Y)
- net SCK_0: now also U1.6 (2Y)
- net SCK_1: now also U1.11 (4Y)
- net VCC: now also C1.1, C2.1, C3.1, C4.1, C5.1, C6.1, C7.1, C8.1, C9.1, C?.1, C?.1, J3.2 (Pin_2), R1.1, R2.1, R3.1, R4.1, R5.1, R6.1, R7.1, R8.1, R9.1, U2.14 (VCC), U3.14 (VCC), U4.14 (VCC)
- net SEL_0: now reaches U1.1 (1~OE)
- net SEL_0: now also U1.4 (2~OE), R1.2
- net SEL_1: now reaches U1.10 (3~OE)
- net SEL_1: now also U1.13 (4~OE), R2.2
- net SCK: now reaches U1.12 (4A)
- net SCK: now also U1.5 (2A), U2.12 (4A), U2.5 (2A), U3.12 (4A), U3.5 (2A), U4.12 (4A), U4.5 (2A)
- net MOSI: now reaches U1.2 (1A)
- net MOSI: now also U1.9 (3A), U2.2 (1A), U2.9 (3A), U3.2 (1A), U3.9 (3A), U4.2 (1A), U4.9 (3A)
- new net: D1.2 (A), R9.2
- new net MOSI_2: U2.3 (1Y)
- new net MOSI_3: U2.8 (3Y)
- new net MOSI_4: U3.3 (1Y)
- new net MOSI_5: U3.8 (3Y)
- new net MOSI_6: U4.3 (1Y)
- new net MOSI_7: U4.8 (3Y)
- new net SCK_2: U2.6 (2Y)
- new net SCK_3: U2.11 (4Y)
- new net SCK_4: U3.6 (2Y)
- new net SCK_5: U3.11 (4Y)
- new net SCK_6: U4.6 (2Y)
- new net SCK_7: U4.11 (4Y)
- new net SEL_2: R3.2, U2.1 (1~OE), U2.4 (2~OE)
- new net SEL_3: R4.2, U2.10 (3~OE), U2.13 (4~OE)
- new net SEL_4: R5.2, U3.1 (1~OE), U3.4 (2~OE)
- new net SEL_5: R6.2, U3.10 (3~OE), U3.13 (4~OE)
- new net SEL_6: R7.2, U4.1 (1~OE), U4.4 (2~OE)
- new net SEL_7: R8.2, U4.10 (3~OE), U4.13 (4~OE)
Other:
- moved on the sheet: J1, J2, U1

Commit message: Schematic complete
Parts:
- added C10, C11: xuF, Capacitor_SMD:C_0603_1608Metric, symbol Device:C_Small
- added J4: SerialConsole_Conn, Connector_PinHeader_2.54mm:PinHeader_1x04_P2.54mm_Vertical, symbol Connector_Generic:Conn_01x04
- added R10, R11: x, Resistor_SMD:R_0201_0603Metric, symbol Device:R_Small
- C1: footprint (none) -> Capacitor_SMD:C_Elec_6.3x5.4; MFG Part No. (none) -> UWT1C101MCL1GB
- C12, C13: renamed from C?; footprint (none) -> Capacitor_SMD:C_0603_1608Metric
- J3: value Screw_Terminal_01x02 -> PWR_Conn; footprint (none) -> GiraffeTech_Terminal.pretty:DINKLE_5EHDRC-2P; MFG Part No. (none) -> 5EHDRC-2P
- U1, U2, U3, U4: footprint (none) -> Package_SO:TSSOP-14_4.4x5mm_P0.65mm
Connections:
- net SEL_0 is gone; now on net GPIO5: R1.2, U1.1 (1~OE), U1.4 (2~OE)
- net SEL_1 is gone; now on net GPIO6: R2.2, U1.10 (3~OE), U1.13 (4~OE)
- net SEL_2 is gone; now on net GPIO12: R3.2, U2.1 (1~OE), U2.4 (2~OE)
- net SEL_3 is gone; now on net GPIO13: R4.2, U2.10 (3~OE), U2.13 (4~OE)
- net SEL_4 is gone; now on net GPIO16: R5.2, U3.1 (1~OE), U3.4 (2~OE)
- net SEL_5 is gone; now on net GPIO19: R6.2, U3.10 (3~OE), U3.13 (4~OE)
- net GND: now also J2.10 (Pin_10), J2.12 (Pin_12), J2.14 (Pin_14), J2.16 (Pin_16), J2.18 (Pin_18), J2.2 (Pin_2), J2.20 (Pin_20), J2.21 (Pin_21), J2.23 (Pin_23), J2.25 (Pin_25), J2.27 (Pin_27), J2.29 (Pin_29), J2.31 (Pin_31), J2.33 (Pin_33), J2.35 (Pin_35), J2.37 (Pin_37), J2.39 (Pin_39), J2.4 (Pin_4), J2.6 (Pin_6), J2.8 (Pin_8), C10.2, C11.2, J4.1 (Pin_1)
- net MOSI: now also J1.19 (Pin_19), C11.1, R11.2
- net MOSI_0: now also J2.5 (Pin_5); no longer J1.19 (Pin_19)
- net MOSI_1: now also J2.9 (Pin_9); no longer J1.38 (Pin_38)
- net MOSI_2: now also J2.13 (Pin_13)
- net MOSI_3: now also J2.17 (Pin_17)
- net MOSI_4: now also J2.22 (Pin_22)
- net MOSI_5: now also J2.26 (Pin_26)
- net MOSI_6: now also J2.30 (Pin_30)
- net MOSI_7: now also J2.34 (Pin_34)
- net RxD: now also J4.3 (Pin_3)
- net SCK: now also J1.23 (Pin_23), C10.1, R10.2
- net SCK_0: now also J2.7 (Pin_7); no longer J1.23 (Pin_23)
- net SCK_1: now also J2.11 (Pin_11); no longer J1.40 (Pin_40)
- net SCK_2: now also J2.15 (Pin_15)
- net SCK_3: now also J2.19 (Pin_19)
- net SCK_4: now also J2.24 (Pin_24)
- net SCK_5: now also J2.28 (Pin_28)
- net SCK_6: now also J2.32 (Pin_32)
- net SCK_7: now also J2.36 (Pin_36)
- net TxD: now also J4.4 (Pin_4)
- net VCC: now also J2.1 (Pin_1), J2.3 (Pin_3), J2.38 (Pin_38), J2.40 (Pin_40), J4.2 (Pin_2), R10.1, R11.1
- net GPIO5: now reaches J1.29 (Pin_29)
- net GPIO6: now reaches J1.31 (Pin_31)
- net GPIO12: now reaches J1.32 (Pin_32)
- net GPIO13: now reaches J1.33 (Pin_33)
- net GPIO16: now reaches J1.36 (Pin_36)
- net GPIO26: now reaches J1.37 (Pin_37)
- net MISO_0 renamed MISO
- net MISO_1 renamed GPIO19
- net SEL_6 renamed GPIO20
- net GPIO20: now also J1.38 (Pin_38)
- net SEL_7 renamed GPIO21
- net GPIO21: now also J1.40 (Pin_40)
- no-connect marks 0 -> 13
Other:
- note added: "OPTIONAL LP-FILTER"
- moved on the sheet: J1, J2

Commit message: Put come more progress
Parts:
- J2: footprint Connector_PinSocket_2.54mm:PinSocket_2x20_P2.54mm_Vertical -> Connector_IDC:IDC-Header_2x20_P2.54mm_Vertical
- J3: footprint GiraffeTech_Terminal.pretty:DINKLE_5EHDRC-2P -> GiraffeTech_Terminal:DINKLE_5EHDRC-2P
- R1, R10, R11, R2, R3, R4, R5, R6, R7, R8, R9: footprint Resistor_SMD:R_0201_0603Metric -> Resistor_SMD:R_0603_1608Metric
Connections:
- net GND: now also J3.2 (Pin_2); no longer J3.1 (Pin_1)
- net VCC: now also J3.1 (Pin_1); no longer J3.2 (Pin_2)
Changed lines of the file:
@@
 F 0 "J2" H 2450 6267 50  0000 C CNN
 F 1 "ExpansionBoard_Conn" H 2450 6176 50  0000 C CNN
-F 2 "Connector_PinSocket_2.54mm:PinSocket_2x20_P2.54mm_Vertical" H 2400 5150 50  0001 C CNN
+F 2 "Connector_IDC:IDC-Header_2x20_P2.54mm_Vertical" H 2400 5150 50  0001 C CNN
 F 3 "~" H 2400 5150 50  0001 C CNN
 	1    2400 5150
@@
 F 0 "R1" V 6004 1650 50  0000 C CNN
 F 1 "10K" V 6095 1650 50  0000 C CNN
-F 2 "Resistor_SMD:R_0201_0603Metric" H 6200 1650 50  0001 C CNN
+F 2 "Resistor_SMD:R_0603_1608Metric" H 6200 1650 50  0001 C CNN
 F 3 "~" H 6200 1650 50  0001 C CNN
 	1    6200 1650
@@
 F 0 "R2" V 6004 1950 50  0000 C CNN
 F 1 "10K" V 6095 1950 50  0000 C CNN
-F 2 "Resistor_SMD:R_0201_0603Metric" H 6200 1950 50  0001 C CNN
+F 2 "Resistor_SMD:R_0603_1608Metric" H 6200 1950 50  0001 C CNN
 F 3 "~" H 6200 1950 50  0001 C CNN
 	1    6200 1950
@@
 F 0 "R3" V 6004 2250 50  0000 C CNN
 F 1 "10K" V 6095 2250 50  0000 C CNN
-F 2 "Resistor_SMD:R_0201_0603Metric" H 6200 2250 50  0001 C CNN
+F 2 "Resistor_SMD:R_0603_1608Metric" H 6200 2250 50  0001 C CNN
 F 3 "~" H 6200 2250 50  0001 C CNN
 	1    6200 2250
@@
 F 0 "R4" V 6004 2550 50  0000 C CNN
 F 1 "10K" V 6095 2550 50  0000 C CNN
-F 2 "Resistor_SMD:R_0201_0603Metric" H 6200 2550 50  0001 C CNN
+F 2 "Resistor_SMD:R_0603_1608Metric" H 6200 2550 50  0001 C CNN
 F 3 "~" H 6200 2550 50  0001 C CNN
 	1    6200 2550
@@
 F 0 "R5" V 6004 2850 50  0000 C CNN
 F 1 "10K" V 6095 2850 50  0000 C CNN
-F 2 "Resistor_SMD:R_0201_0603Metric" H 6200 2850 50  0001 C CNN
+F 2 "Resistor_SMD:R_0603_1608Metric" H 6200 2850 50  0001 C CNN
 F 3 "~" H 6200 2850 50  0001 C CNN
 	1    6200 2850
@@
 F 0 "R6" V 6004 3150 50  0000 C CNN
 F 1 "10K" V 6095 3150 50  0000 C CNN
-F 2 "Resistor_SMD:R_0201_0603Metric" H 6200 3150 50  0001 C CNN
+F 2 "Resistor_SMD:R_0603_1608Metric" H 6200 3150 50  0001 C CNN
 F 3 "~" H 6200 3150 50  0001 C CNN
 	1    6200 3150
@@
 F 0 "R7" V 6004 3450 50  0000 C CNN
 F 1 "10K" V 6095 3450 50  0000 C CNN
-F 2 "Resistor_SMD:R_0201_0603Metric" H 6200 3450 50  0001 C CNN
+F 2 "Resistor_SMD:R_0603_1608Metric" H 6200 3450 50  0001 C CNN
 F 3 "~" H 6200 3450 50  0001 C CNN
 	1    6200 3450
@@
 F 0 "R8" V 6004 3750 50  0000 C CNN
 F 1 "10K" V 6095 3750 50  0000 C CNN
-F 2 "Resistor_SMD:R_0201_0603Metric" H 6200 3750 50  0001 C CNN
+F 2 "Resistor_SMD:R_0603_1608Metric" H 6200 3750 50  0001 C CNN
 F 3 "~" H 6200 3750 50  0001 C CNN
 	1    6200 3750
@@
 L Connector:Screw_Terminal_01x02 J3
 U 1 1 5CC76F3F
-P 4600 5200
-F 0 "J3" H 4520 4875 50  0000 C CNN
-F 1 "PWR_Conn" H 4520 4966 50  0000 C CNN
-F 2 "GiraffeTech_Terminal.pretty:DINKLE_5EHDRC-2P" H 4600 5200 50  0001 C CNN
-F 3 "~" H 4600 5200 50  0001 C CNN
-F 4 "5EHDRC-2P" H 4600 5200 50  0001 C CNN "MFG Part No."
-	1    4600 5200
-	-1   0    0    1
+P 4600 5100
+F 0 "J3" H 4600 5350 50  0000 C CNN
+F 1 "PWR_Conn" H 4600 5250 50  0000 C CNN
+F 2 "GiraffeTech_Terminal:DINKLE_5EHDRC-2P" H 4600 5100 50  0001 C CNN
+F 3 "~" H 4600 5100 50  0001 C CNN
+F 4 "5EHDRC-2P" H 4600 5100 50  0001 C CNN "MFG Part No."
+	1    4600 5100
+	-1   0    0    -1
 $EndComp
 $Comp
@@
 	0    1    1    0
 $EndComp
-Wire Wire Line
-	4800 5100 4900 5100
 $Comp
 L Device:CP1_Small C1
@@
 F 0 "R9" H 4959 6096 50  0000 L CNN
 F 1 "1K" H 4959 6005 50  0000 L CNN
-F 2 "Resistor_SMD:R_0201_0603Metric" H 4900 6050 50  0001 C CNN
+F 2 "Resistor_SMD:R_0603_1608Metric" H 4900 6050 50  0001 C CNN
 F 3 "~" H 4900 6050 50  0001 C CNN
 	1    4900 6050
@@
 F 0 "R10" H 3809 2146 50  0000 L CNN
 F 1 "x" H 3809 2055 50  0000 L CNN
-F 2 "Resistor_SMD:R_0201_0603Metric" H 3750 2100 50  0001 C CNN
+F 2 "Resistor_SMD:R_0603_1608Metric" H 3750 2100 50  0001 C CNN
 F 3 "~" H 3750 2100 50  0001 C CNN
 	1    3750 2100
@@
 F 0 "R11" H 4209 2146 50  0000 L CNN
 F 1 "x" H 4209 2055 50  0000 L CNN
-F 2 "Resistor_SMD:R_0201_0603Metric" H 4150 2100 50  0001 C CNN
+F 2 "Resistor_SMD:R_0603_1608Metric" H 4150 2100 50  0001 C CNN
 F 3 "~" H 4150 2100 50  0001 C CNN
 	1    4150 2100
@@
 	2700 6150 3200 6150
 $Comp
-L power:GND #PWR?
+L power:GND #PWR0156
 U 1 1 5D247061
 P 1700 6250
-F 0 "#PWR?" H 1700 6000 50  0001 C CNN
+F 0 "#PWR0156" H 1700 6000 50  0001 C CNN
 F 1 "GND" H 1705 6077 50  0000 C CNN
 F 2 "" H 1700 6250 50  0001 C CNN
@@
 	1700 6150 1700 6250
 $Comp
-L power:GND #PWR?
+L power:GND #PWR0157
 U 1 1 5D25CE88
 P 3200 4150
-F 0 "#PWR?" H 3200 3900 50  0001 C CNN
+F 0 "#PWR0157" H 3200 3900 50  0001 C CNN
 F 1 "GND" H 3205 3977 50  0000 C CNN
 F 2 "" H 3200 4150 50  0001 C CNN
@@
 	3200 5050 3200 5150
 $Comp
-L power:VCC #PWR?
+L power:VCC #PWR0158
 U 1 1 5D273E25
 P 1700 4150
-F 0 "#PWR?" H 1700 4000 50  0001 C CNN
+F 0 "#PWR0158" H 1700 4000 50  0001 C CNN
 F 1 "VCC" H 1717 4323 50  0000 C CNN
 F 2 "" H 1700 4150 50  0001 C CNN
@@
 	1700 4250 1700 4350
 $Comp
-L power:VCC #PWR?
+L power:VCC #PWR0159
 U 1 1 5D28BCDC
 P 3200 6250
-F 0 "#PWR?" H 3200 6100 50  0001 C CNN
+F 0 "#PWR0159" H 3200 6100 50  0001 C CNN
 F 1 "VCC" H 3218 6423 50  0000 C CNN
 F 2 "" H 3200 6250 50  0001 C CNN
@@
 NoConn ~ 2700 3100
 NoConn ~ 2200 3100
+Wire Wire Line
+	4800 5100 4900 5100
 $EndSCHEMATC

Commit message: Push more effort
Parts:
- removed J4: SerialConsole_Conn, Connector_PinHeader_2.54mm:PinHeader_1x04_P2.54mm_Vertical, symbol Connector_Generic:Conn_01x04
Connections:
- net GND: now also J2.11 (Pin_11), J2.13 (Pin_13), J2.15 (Pin_15), J2.17 (Pin_17), J2.19 (Pin_19), J2.5 (Pin_5), J2.7 (Pin_7), J2.9 (Pin_9); no longer J2.10 (Pin_10), J2.12 (Pin_12), J2.14 (Pin_14), J2.16 (Pin_16), J2.18 (Pin_18), J2.20 (Pin_20), J2.6 (Pin_6), J2.8 (Pin_8)
- net GPIO20: no longer R7.2, U4.1 (1~OE), U4.4 (2~OE)
- net GPIO26: now also R7.2, U4.1 (1~OE), U4.4 (2~OE)
- net MOSI_0: now also J2.6 (Pin_6); no longer J2.5 (Pin_5)
- net MOSI_1: now also J2.10 (Pin_10); no longer J2.9 (Pin_9)
- net MOSI_2: now also J2.14 (Pin_14); no longer J2.13 (Pin_13)
- net MOSI_3: now also J2.18 (Pin_18); no longer J2.17 (Pin_17)
- net SCK_0: now also J2.8 (Pin_8); no longer J2.7 (Pin_7)
- net SCK_1: now also J2.12 (Pin_12); no longer J2.11 (Pin_11)
- net SCK_2: now also J2.16 (Pin_16); no longer J2.15 (Pin_15)
- net SCK_3: now also J2.20 (Pin_20); no longer J2.19 (Pin_19)

Commit message: A little bit closer to the final
Connections:
- net GND: now also J2.38 (Pin_38), J2.40 (Pin_40); no longer J2.2 (Pin_2), J2.4 (Pin_4)
- net VCC: now also J2.2 (Pin_2), J2.4 (Pin_4); no longer J2.38 (Pin_38), J2.40 (Pin_40)
- net +3V3: no longer names the net of J1.1 (Pin_1)
- net +3V3: no longer J1.17 (Pin_17)
- no-connect marks 13 -> 15
Changed lines of the file:
@@
 	2000 3500 2200 3500
-$Comp
-L power:+3.3V #PWR0109
-U 1 1 5CBD8CCF
-P 2000 1700
-F 0 "#PWR0109" H 2000 1550 50  0001 C CNN
-F 1 "+3.3V" H 2015 1873 50  0000 C CNN
-F 2 "" H 2000 1700 50  0001 C CNN
-F 3 "" H 2000 1700 50  0001 C CNN
-	1    2000 1700
-	1    0    0    -1
-$EndComp
-Wire Wire Line
-	2000 1700 2000 1800
-Wire Wire Line
-	2000 1800 2100 1800
 $Comp
 L InGarage_Logic_LevelTranslator:SN74LV4T125 U1
@@
 Wire Wire Line
 	6350 5250 6350 5350
-Wire Wire Line
-	2200 2600 2100 2600
-Wire Wire Line
-	2100 2600 2100 1800
-Connection ~ 2100 1800
-Wire Wire Line
-	2100 1800 2200 1800
 $Comp
 L Device:C_Small C10
@@
 SCK_2
 Wire Wire Line
-	1700 4250 2200 4250
-Wire Wire Line
-	1700 4350 2200 4350
-Wire Wire Line
 	1700 5250 2200 5250
 Wire Wire Line
@@
 Wire Wire Line
 	2700 4350 3200 4350
-Wire Wire Line
-	2700 6050 3200 6050
-Wire Wire Line
-	2700 6150 3200 6150
 $Comp
 L power:GND #PWR0156
@@
 Wire Wire Line
 	1700 6150 1700 6250
-$Comp
-L power:GND #PWR0157
-U 1 1 5D25CE88
-P 3200 4150
-F 0 "#PWR0157" H 3200 3900 50  0001 C CNN
-F 1 "GND" H 3205 3977 50  0000 C CNN
-F 2 "" H 3200 4150 50  0001 C CNN
-F 3 "" H 3200 4150 50  0001 C CNN
-	1    3200 4150
-	-1   0    0    1
-$EndComp
 Wire Wire Line
 	3200 4150 3200 4250
@@
 Wire Wire Line
 	3200 4250 3200 4350
-$Comp
-L power:VCC #PWR0158
-U 1 1 5D273E25
-P 1700 4150
-F 0 "#PWR0158" H 1700 4000 50  0001 C CNN
-F 1 "VCC" H 1717 4323 50  0000 C CNN
-F 2 "" H 1700 4150 50  0001 C CNN
-F 3 "" H 1700 4150 50  0001 C CNN
-	1    1700 4150
-	1    0    0    -1
-$EndComp
-Wire Wire Line
-	1700 4150 1700 4250
-Connection ~ 1700 4250
-Wire Wire Line
-	1700 4250 1700 4350
-$Comp
-L power:VCC #PWR0159
-U 1 1 5D28BCDC
-P 3200 6250
-F 0 "#PWR0159" H 3200 6100 50  0001 C CNN
-F 1 "VCC" H 3218 6423 50  0000 C CNN
-F 2 "" H 3200 6250 50  0001 C CNN
-F 3 "" H 3200 6250 50  0001 C CNN
-	1    3200 6250
-	-1   0    0    1
-$EndComp
-Wire Wire Line
-	3200 6050 3200 6150
-Connection ~ 3200 6150
-Wire Wire Line
-	3200 6150 3200 6250
 NoConn ~ 2200 2100
 NoConn ~ 2200 2300
@@
 Wire Wire Line
 	1700 5150 1700 5050
+$Comp
+L power:VCC #PWR0109
+U 1 1 5CC9E623
+P 1700 4150
+F 0 "#PWR0109" H 1700 4000 50  0001 C CNN
+F 1 "VCC" H 1717 4323 50  0000 C CNN
+F 2 "" H 1700 4150 50  0001 C CNN
+F 3 "" H 1700 4150 50  0001 C CNN
+	1    1700 4150
+	1    0    0    -1
+$EndComp
+Wire Wire Line
+	1700 4150 1700 4250
+Wire Wire Line
+	1700 4350 2200 4350
+Wire Wire Line
+	2200 4250 1700 4250
+Connection ~ 1700 4250
+Wire Wire Line
+	1700 4250 1700 4350
+$Comp
+L power:VCC #PWR0154
+U 1 1 5CCC81E0
+P 3200 4150
+F 0 "#PWR0154" H 3200 4000 50  0001 C CNN
+F 1 "VCC" H 3217 4323 50  0000 C CNN
+F 2 "" H 3200 4150 50  0001 C CNN
+F 3 "" H 3200 4150 50  0001 C CNN
+	1    3200 4150
+	1    0    0    -1
+$EndComp
+$Comp
+L power:GND #PWR0155
+U 1 1 5CCC8970
+P 3200 6250
+F 0 "#PWR0155" H 3200 6000 50  0001 C CNN
+F 1 "GND" H 3205 6077 50  0000 C CNN
+F 2 "" H 3200 6250 50  0001 C CNN
+F 3 "" H 3200 6250 50  0001 C CNN
+	1    3200 6250
+	1    0    0    -1
+$EndComp
+Wire Wire Line
+	2700 6050 3200 6050
+Wire Wire Line
+	3200 6050 3200 6150
+Wire Wire Line
+	2700 6150 3200 6150
+Connection ~ 3200 6150
+Wire Wire Line
+	3200 6150 3200 6250
+NoConn ~ 2200 1800
+NoConn ~ 2200 2600
 $EndSCHEMATC
